File: D23.kicad_pcb (KiCad board)
At the start: 6 copper layers, 19 x 13 mm, 61 parts, among them IC1 AVR64DD28-I_STX, IC2 NCP730BM, IC3 DRV8231ADSGR, J1 Conn_02x0_Counter_Clockwise, J10 AUX4.od, J11 Conn_01x01, J12 VHBR, J2 Conn_01x01, J3 AUX1.od, J4 AUX2.od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

Commit message: add: fuses
Parts:
- J1: value Conn_02x0_Counter_Clockwise -> NEM 652
- R13: value 3.3k -> 1k
- R16, R18: value 10k -> 12k

Commit message: updated Kicad version
Other:
- net class Default removed
- net class Power removed
